File: schematics/Main_board/Main_board/Main_board.kicad_sch (KiCad schematic)
At the start: 36 parts, among them J1 USB_B_Micro, J2 Conn_01x16_Female, J3 TOUCH, Q1 UMH3N, U1 ESP32-S3-WROOM-1, U2 AP2112K-3.3, U3 BQ21040DBVR, U4 CH340G, U5 PCF8563T, U6 LCD, U7 LSM6DS3, Y1 12Mhz, Y2 32.768kHz

Commit message: Update: First pcb revision complete
Parts:
- removed J3: TOUCH, LCD:slide_sensor_8p, symbol Connector:Conn_01x08_Female
- removed U3: BQ21040DBVR, Package_TO_SOT_SMD:SOT-23-6, symbol Battery_Management:AP9101CK6
- removed Y1: 12Mhz, Crystal:Resonator_SMD_Murata_CSTxExxV-3Pin_3.0x1.1mm_HandSoldering, symbol Device:Crystal
- added H1, H2, H3, H4: MountingHole, MountingHole:MountingHole_3.5mm_Pad_Via, symbol Mechanical:MountingHole
- added H5, H6, H7, H8: MountingHole, MountingHole:MountingHole_2.2mm_M2_DIN965, symbol Mechanical:MountingHole
- added J3, J5: Conn_01x06_Female, LCD:slider_sensors_points_smd, symbol Connector:Conn_01x06_Female
- added J4: Conn_01x06_Female, LCD:slide_sensor_6p, symbol Connector:Conn_01x06_Female
- added R6: 1K, Resistor_SMD:R_0201_0603Metric_Pad0.64x0.40mm_HandSolder, symbol Device:R
- added U3: bq21040, Package_TO_SOT_SMD:SOT-23-6_Handsoldering, symbol LCD_IIC_12864:bq21040
- added Y1: Crystal_GND2_Small, Crystal:Resonator_SMD_Murata_CSTxExxV-3Pin_3.0x1.1mm_HandSoldering, symbol Device:Crystal_GND2_Small
- BT2: footprint (none) -> LCD:lipo_battery_800mA
- C4, C5: Place (none) -> NC
- C8: value 8p -> 22p
- R3: value 120 -> 1k5
Connections:
- net NCH_CH_PIN is gone; now on net +BATT: R3.2
- net +3V3: now also U7.12 (CS)
- net +5V: now also C3.2, U3.6 (VIN)
- net +BATT: now also BT2.1 (+), C9.2, U3.2 (VOUT)
- net GNDREF: now also C3.1, C9.1, R6.2, U3.5 (GND), Y1.2; no longer C3.2, D1.1 (K)
- net I/O_1: now also J2.3 (Pin_3); no longer J2.10 (Pin_10)
- net I/O_2: now also J2.4 (Pin_4); no longer J2.11 (Pin_11)
- net I/O_3: now also J2.5 (Pin_5); no longer J2.12 (Pin_12)
- net I/O_4: now also J2.6 (Pin_6); no longer J2.13 (Pin_13)
- net I/O_5: now also J2.7 (Pin_7); no longer J2.14 (Pin_14)
- net MISO: now also J2.13 (Pin_13); no longer J2.6 (Pin_6)
- net MOSI: now also J2.12 (Pin_12); no longer J2.5 (Pin_5)
- net SCL_1: now also J2.11 (Pin_11); no longer J2.9 (Pin_9)
- net SDA_1: now also J2.10 (Pin_10); no longer J2.8 (Pin_8)
- net SPI_CLK: now also J2.14 (Pin_14); no longer J2.7 (Pin_7)
- net TOUCH_1: now also J3.1 (Pin_1); no longer U1.22 (GPIO14/TOUCH14/ADC2_CH3/FSPIWP/FSPIDQS/SUBSPIWP)
- net TOUCH_2: now also J3.2 (Pin_2)
- net TOUCH_3: now also J3.3 (Pin_3)
- net TOUCH_4: now also J3.4 (Pin_4)
- net TOUCH_5: now also J3.5 (Pin_5)
- net UART_RX: now also J2.9 (Pin_9); no longer J2.4 (Pin_4)
- net UART_TX: now also J2.8 (Pin_8); no longer J2.3 (Pin_3)
- net at C4.1, U4.8 (XO): now also Y1.1
- net at C5.1, U4.7 (XI): now also Y1.3
- net at TH1.1: now also U3.1 (TS)
- removed net +3.3V: BT2.1 (+), C9.1, U7.12 (CS)
- new net: J4.1 (Pin_1), J5.1 (Pin_1)
- new net: J4.2 (Pin_2), J5.2 (Pin_2)
- new net: J4.3 (Pin_3), J5.3 (Pin_3)
- new net: J4.4 (Pin_4), J5.4 (Pin_4)
- new net: J4.5 (Pin_5), J5.5 (Pin_5)
- new net: J4.6 (Pin_6), J5.6 (Pin_6)
- new net: R6.1, U3.4 (ISET)
- new net: D1.1 (K), U3.3 (CHR)
- new net TOUCH_6: J3.6 (Pin_6), U1.22 (GPIO14/TOUCH14/ADC2_CH3/FSPIWP/FSPIDQS/SUBSPIWP)
Other:
- note added: "- Add short circuit protection - Make test circuit before conect MCU - Add adc for battery state"
- note added: "Charging current to 540mA R_iset=K_iset/I_out R_iset=540Aohms/540mA R_iset=1K"
- note removed: "- Add short circuit protection - Make test circuit before conect MCU - Add ESD Protection - Create new extended footprint for LIS3DH - Add adc for battery state"
- moved on the sheet: BT2, C3, C9, D1, R3, TH1

Commit message: update: to kicad version 7, and arrange all the components on their respective hierarchy page
Parts:
- removed BT1: 1v5 LR44, LCD:MY-LR44-02, symbol Device:Battery_Cell
- removed BT2: 3v7 LIpo, LCD:lipo_battery_800mA, symbol Device:Battery_Cell
- removed C1, C2, C3, C9: 1uf, Capacitor_SMD:C_0201_0603Metric, symbol Device:C
- removed C10, C11: 100nf, Capacitor_SMD:C_0201_0603Metric, symbol Device:C
- removed C8: 22p, Capacitor_SMD:C_0201_0603Metric, symbol Device:C
- removed D1: LED, LED_SMD:LED_0402_1005Metric_Pad0.77x0.64mm_HandSolder, symbol Device:LED
- removed D2, D3, D4: 0603ESDA-05N, Resistor_SMD:R_0603_1608Metric, symbol Device:D_TVS
- removed H1, H2, H3, H4: MountingHole, MountingHole:MountingHole_3.5mm_Pad_Via, symbol Mechanical:MountingHole
- removed H5, H6, H7, H8: MountingHole, MountingHole:MountingHole_2.2mm_M2_DIN965, symbol Mechanical:MountingHole
- removed J1: USB_B_Micro, Connector_USB:USB_Micro-B_Amphenol_10118194_Horizontal, symbol Connector:USB_B_Micro
- removed J2: Conn_01x16_Female, Connector_PinSocket_2.54mm:PinSocket_1x16_P2.54mm_Horizontal, symbol Connector:Conn_01x16_Female
- removed J3, J5: Conn_01x06_Female, LCD:slider_sensors_points_smd, symbol Connector:Conn_01x06_Female
- removed J4: Conn_01x06_Female, LCD:slide_sensor_6p, symbol Connector:Conn_01x06_Female
- removed R3: 1k5, Resistor_SMD:R_0201_0603Metric_Pad0.64x0.40mm_HandSolder, symbol Device:R
- removed R4, R5: 4k7, Resistor_SMD:R_0603_1608Metric_Pad0.98x0.95mm_HandSolder, symbol Device:R
- removed R6: 1K, Resistor_SMD:R_0201_0603Metric_Pad0.64x0.40mm_HandSolder, symbol Device:R
- removed TH1: NCP18XH103F03RB, Resistor_SMD:R_0603_1608Metric, symbol Device:Thermistor_NTC
- removed U2: AP2112K-3.3, Package_TO_SOT_SMD:SOT-23-5, symbol Regulator_Linear:AP2112K-3.3
- removed U3: bq21040, Package_TO_SOT_SMD:SOT-23-6_Handsoldering, symbol LCD_IIC_12864:bq21040
- removed U5: PCF8563T, Package_SO:SOIC-8_3.9x4.9mm_P1.27mm, symbol Timer_RTC:PCF8563T
- removed U6: LCD, LCD:LCD_IIC_12864, symbol LCD_IIC_12864:LCD
- removed U7: LSM6DS3, Package_LGA:LGA-14_3x2.5mm_P0.5mm_LayoutBorder3x4y, symbol Sensor_Motion:LSM6DS3
- removed Y2: 32.768kHz, Crystal:Crystal_C38-LF_D3.0mm_L8.0mm_Horizontal, symbol Device:Crystal
Other:
- added sheet Connectors (connectors.kicad_sch)
- added sheet Peripherals (Sensors.kicad_sch)
- added sheet Power (power.kicad_sch)
- note removed: "3.3v Power Regulator"
- note removed: "Attitude Sensor/Gyroscope"
- note removed: "Battery management system"
- note removed: "Charging current to 540mA R_iset=K_iset/I_out R_iset=540Aohms/540mA R_iset=1K"
- note removed: "GPIO & Communication peripherals"
- note removed: "LCD Screen 128x64"
- note removed: "MicroUSB_Connection"
- note removed: "Real Time clock"
- note removed: "SDO/SA0 pin is connected to ground, the LSb value is '0' (address 1101010b)"
- note removed: "Slider sensor Capacitive buttons"
- note removed: "i2c Pull-up resistors"
- moved on the sheet: C4, C5, C6, C7, Q1A, Q1B, R1, R2, U4, Y1

Commit message: fix: 3d step file paths
Parts:
- C4, C5, C6, C7: footprint Capacitor_SMD:C_0201_0603Metric -> Capacitor_SMD:C_0402_1005Metric
- R1, R2: footprint Resistor_SMD:R_0201_0603Metric_Pad0.64x0.40mm_HandSolder -> Resistor_SMD:R_0402_1005Metric
Changed lines of the file:
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@@
       (effects (font (size 1.27 1.27)) (justify left))
     )
-    (property "Footprint" "Capacitor_SMD:C_0201_0603Metric" (at 29.4132 179.07 0)
+    (property "Footprint" "Capacitor_SMD:C_0402_1005Metric" (at 29.4132 179.07 0)
       (effects (font (size 1.27 1.27)) hide)
     )
@@
       (effects (font (size 1.27 1.27)))
     )
-    (property "Footprint" "Capacitor_SMD:C_0201_0603Metric" (at 47.625 140.0048 0)
+    (property "Footprint" "Capacitor_SMD:C_0402_1005Metric" (at 47.625 140.0048 0)
       (effects (font (size 1.27 1.27)) hide)
     )
@@
       (effects (font (size 1.27 1.27)))
     )
-    (property "Footprint" "Capacitor_SMD:C_0201_0603Metric" (at 59.055 140.0048 0)
+    (property "Footprint" "Capacitor_SMD:C_0402_1005Metric" (at 59.055 140.0048 0)
       (effects (font (size 1.27 1.27)) hide)
     )
@@
       (effects (font (size 1.27 1.27)) (justify left))
     )
-    (property "Footprint" "Resistor_SMD:R_0201_0603Metric_Pad0.64x0.40mm_HandSolder" (at 83.947 177.8 90)
+    (property "Footprint" "Resistor_SMD:R_0402_1005Metric" (at 83.947 177.8 90)
       (effects (font (size 1.27 1.27)) hide)
     )
@@
       (effects (font (size 1.27 1.27)) (justify left))
     )
-    (property "Footprint" "Capacitor_SMD:C_0201_0603Metric" (at 39.7002 179.07 0)
+    (property "Footprint" "Capacitor_SMD:C_0402_1005Metric" (at 39.7002 179.07 0)
       (effects (font (size 1.27 1.27)) hide)
     )
@@
       (effects (font (size 1.27 1.27)) (justify left))
     )
-    (property "Footprint" "Resistor_SMD:R_0201_0603Metric_Pad0.64x0.40mm_HandSolder" (at 102.362 171.45 90)
-      (effects (font (size 1.27 1.27)) hide)
-    )
+    (property "Footprint" "Resistor_SMD:R_0402_1005Metric" (at 102.362 171.45 90)
+      (effects (font (size 1.27 1.27)) hide)
+    )
