File: schematics/Main_board/Main_board/power.kicad_sch (KiCad schematic)
At the start: 11 parts, among them U2 AP2112K-3.3, U3 bq21040

Commit message: fix: 3d step file paths
Parts:
- C1, C2, C3, C9: footprint Capacitor_SMD:C_0201_0603Metric -> Capacitor_SMD:C_0402_1005Metric
- R3, R6: footprint Resistor_SMD:R_0201_0603Metric_Pad0.64x0.40mm_HandSolder -> Resistor_SMD:R_0402_1005Metric
Changed lines of the file:
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@@
       (effects (font (size 1.27 1.27)) (justify left))
     )
-    (property "Footprint" "Resistor_SMD:R_0201_0603Metric_Pad0.64x0.40mm_HandSolder" (at 33.782 40.64 90)
+    (property "Footprint" "Resistor_SMD:R_0402_1005Metric" (at 33.782 40.64 90)
       (effects (font (size 1.27 1.27)) hide)
     )
@@
       (effects (font (size 1.27 1.27)) (justify right))
     )
-    (property "Footprint" "Capacitor_SMD:C_0201_0603Metric" (at 91.7448 34.29 0)
+    (property "Footprint" "Capacitor_SMD:C_0402_1005Metric" (at 91.7448 34.29 0)
       (effects (font (size 1.27 1.27)) hide)
     )
@@
       (effects (font (size 1.27 1.27)) (justify right))
     )
-    (property "Footprint" "Resistor_SMD:R_0201_0603Metric_Pad0.64x0.40mm_HandSolder" (at 83.058 38.1 90)
+    (property "Footprint" "Resistor_SMD:R_0402_1005Metric" (at 83.058 38.1 90)
       (effects (font (size 1.27 1.27)) hide)
     )
@@
       (effects (font (size 1.27 1.27)) (justify left))
     )
-    (property "Footprint" "Capacitor_SMD:C_0201_0603Metric" (at 27.6352 83.82 0)
+    (property "Footprint" "Capacitor_SMD:C_0402_1005Metric" (at 27.6352 83.82 0)
       (effects (font (size 1.27 1.27)) hide)
     )
@@
       (effects (font (size 1.27 1.27)) (justify right))
     )
-    (property "Footprint" "Capacitor_SMD:C_0201_0603Metric" (at 26.9748 34.29 0)
+    (property "Footprint" "Capacitor_SMD:C_0402_1005Metric" (at 26.9748 34.29 0)
       (effects (font (size 1.27 1.27)) hide)
     )
@@
       (effects (font (size 1.27 1.27)) (justify left))
     )
-    (property "Footprint" "Capacitor_SMD:C_0201_0603Metric" (at 58.1152 83.82 0)
-      (effects (font (size 1.27 1.27)) hide)
-    )
+    (property "Footprint" "Capacitor_SMD:C_0402_1005Metric" (at 58.1152 83.82 0)
+      (effects (font (size 1.27 1.27)) hide)
+    )
